File: PCB/Fossa PCB.kicad_sch (KiCad schematic)
At the start: 9 parts, among them J1 WT32-SC01, J2 NV10USB+, J3 DG600F, J4 Barrel_Jack_MountingPin, J5 IN+, J6 IN-, J7 OUT+, J8 OUT-, J9 Printer

Commit message: Added Wiring diagram and organised docs a bit
Connections:
- net at J9.3 (Pin_3): now also J1.20 (Pin_20); no longer J1.25 (Pin_25)
- net at J9.4 (Pin_4): now also J1.22 (Pin_22); no longer J1.27 (Pin_27)
Changed lines of the file:
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@@
+    (stroke (width 0) (type default))
+  )
+  (wire (pts (xy 238.76 121.92) (xy 238.76 74.93))
+    (stroke (width 0) (type default))
+  )
+  (wire (pts (xy 241.3 78.74) (xy 208.28 78.74))
     (stroke (width 0) (type default))
   )
@@
     (stroke (width 0) (type default))
   )
+  (wire (pts (xy 241.3 124.46) (xy 241.3 78.74))
+    (stroke (width 0) (type default))
+  )
+  (wire (pts (xy 208.28 78.74) (xy 208.28 85.09))
+    (stroke (width 0) (type default))
+  )
   (wire (pts (xy 135.89 63.5) (xy 146.05 63.5))
     (stroke (width 0) (type default))
@@
   )
   (wire (pts (xy 125.73 57.15) (xy 125.73 93.98))
+    (stroke (width 0) (type default))
+  )
+  (wire (pts (xy 205.74 74.93) (xy 205.74 85.09))
     (stroke (width 0) (type default))
   )
@@
     (stroke (width 0) (type default))
   )
-  (wire (pts (xy 213.36 121.92) (xy 213.36 97.79))
-    (stroke (width 0) (type default))
-  )
   (wire (pts (xy 107.95 120.65) (xy 121.92 120.65))
     (stroke (width 0) (type default))
@@
     (stroke (width 0) (type default))
   )
-  (wire (pts (xy 243.84 121.92) (xy 213.36 121.92))
-    (stroke (width 0) (type default))
-  )
   (wire (pts (xy 234.95 71.12) (xy 214.63 71.12))
     (stroke (width 0) (type default))
@@
     (stroke (width 0) (type default))
   )
+  (wire (pts (xy 243.84 121.92) (xy 238.76 121.92))
+    (stroke (width 0) (type default))
+  )
   (wire (pts (xy 187.96 111.76) (xy 187.96 97.79))
+    (stroke (width 0) (type default))
+  )
+  (wire (pts (xy 238.76 74.93) (xy 205.74 74.93))
     (stroke (width 0) (type default))
   )
@@
   )
   (wire (pts (xy 111.76 66.04) (xy 111.76 81.28))
-    (stroke (width 0) (type default))
-  )
-  (wire (pts (xy 215.9 97.79) (xy 215.9 124.46))
     (stroke (width 0) (type default))
   )
@@
     (stroke (width 0) (type default))
   )
-  (wire (pts (xy 215.9 124.46) (xy 243.84 124.46))
-    (stroke (width 0) (type default))
-  )
   (wire (pts (xy 218.44 134.62) (xy 218.44 97.79))
     (stroke (width 0) (type default))
@@
     (stroke (width 0) (type default))
   )
+  (wire (pts (xy 243.84 124.46) (xy 241.3 124.46))
+    (stroke (width 0) (type default))
+  )
